Commit message: 车轮电机使用JointEffortController驱动成功

File: wheel-leg_ws/src/wheel_leg3/urdf/wheel_leg3.xacro (robot description, xacro)
@@ -7,4 +7,12 @@
   <!-- Import all Gazebo-customization elements, including Gazebo colors -->
   <xacro:include filename="$(find wheel_leg3)/urdf/wheel_leg3.gazebo" />
+  <link name="dummy" />
+  <joint name="joint_dummy_base_link" type="fixed">
+  <origin
+      xyz="0 0 0.253"
+      rpy="0 0 0" />
+    <parent link="dummy" />
+    <child link="base_link" />
+  </joint>
   <link
     name="base_link">
@@ -15,5 +23,5 @@
       <mass
         value="3.0" />
-      <inertia
+      <!-- <inertia
         ixx="0.004712"
         ixy="-9.6242E-20"
@@ -21,6 +29,6 @@
         iyy="0.02081558"
         iyz="-2.8504E-20"
-        izz="0.017536" />
-      <!-- <inertia
+        izz="0.017536" /> -->
+      <inertia
         ixx="0.02763116"
         ixy="-9.6242E-20"
@@ -28,5 +36,5 @@
         iyy="0.009424"
         iyz="-2.8504E-20"
-        izz="0.035072" /> -->
+        izz="0.035072" />
     </inertial>
     <visual>
@@ -272,5 +280,5 @@
     <dynamics damping="0.1" friction="0.0"/>
   </joint>
-  <!-- <transmission name="tran1">
+  <transmission name="tran1">
     <type>transmission_interface/SimpleTransmission</type>
     <joint name="joint_leg1_wheel1">
@@ -291,4 +299,4 @@
       <mechanicalReduction>1</mechanicalReduction>
     </actuator>
-  </transmission> -->
+  </transmission>
 </robot>
