Commit message: 增加imu_link和IMU Sensor

File: wheel-leg_ws/src/wheel_leg3/urdf/wheel_leg3_dae.xacro (robot description, xacro)
@@ -251,4 +251,11 @@
     <dynamics damping="0.1" friction="0.0"/>
   </joint>
+  <link name="imu_link"/>
+  <joint name="base_to_imu" type="fixed">
+    <axis rpy="0 0 0" xyz="0 0 0"/>
+    <parent link="base_link"/>
+    <child link="imu_link"/>
+    <origin rpy="0 0 0" xyz="0 0 0.04"/>
+  </joint>
   <transmission name="tran1">
     <type>transmission_interface/SimpleTransmission</type>

File: wheel-leg_ws/src/wheel_leg3/urdf/wheel_leg3_stl.xacro (robot description, xacro)
@@ -279,4 +279,11 @@
       xyz="0 1 0" />
     <dynamics damping="0.1" friction="0.0"/>
+  </joint>
+  <link name="imu_link"/>
+  <joint name="base_to_imu" type="fixed">
+    <axis rpy="0 0 0" xyz="0 0 0"/>
+    <parent link="base_link"/>
+    <child link="imu_link"/>
+    <origin rpy="0 0 0" xyz="0 0 0.04"/>
   </joint>
   <transmission name="tran1">

Commit message: 在launch文件里指定参数启动odom->tf脚本

File: wheel-leg_ws/src/wheel_leg3/urdf/wheel_leg3_dae.xacro (robot description, xacro)
@@ -7,10 +7,10 @@
   <!-- Import all Gazebo-customization elements, including Gazebo colors -->
   <xacro:include filename="$(find wheel_leg3)/urdf/wheel_leg3.gazebo" />
-  <link name="dummy" />
-  <joint name="joint_dummy_base_link" type="fixed">
+  <link name="base_footprint" />
+  <joint name="joint_base_footprint_base_link" type="fixed">
   <origin
       xyz="0 0 0.253"
       rpy="0 0 0" />
-    <parent link="dummy" />
+    <parent link="base_footprint" />
     <child link="base_link" />
   </joint>
@@ -46,4 +46,9 @@
           filename="package://wheel_leg3/meshes/base_link.dae" />
       </geometry>
+      <material
+        name="">
+        <color
+          rgba="0.90588 0.39607 0.101960 1" />
+      </material>
     </visual>
     <collision>
@@ -81,4 +86,9 @@
           filename="package://wheel_leg3/meshes/link_leg1.dae" />
       </geometry>
+      <material
+        name="">
+        <color
+          rgba="0.79216 0.81961 0.93333 1" />
+      </material>
     </visual>
     <collision>
@@ -129,4 +139,9 @@
           filename="package://wheel_leg3/meshes/link_wheel1.dae" />
       </geometry>
+      <material
+        name="">
+        <color
+          rgba="0.79216 0.81961 0.93333 1" />
+      </material>
     </visual>
     <collision>
@@ -151,5 +166,5 @@
       link="link_wheel1" />
     <axis
-      xyz="0 -1 0" />
+      xyz="0 1 0" />
     <dynamics damping="0.1" friction="0.0"/>
   </joint>
@@ -178,4 +193,9 @@
           filename="package://wheel_leg3/meshes/link_leg2.dae" />
       </geometry>
+      <material
+        name="">
+        <color
+          rgba="0.79216 0.81961 0.93333 1" />
+      </material>
     </visual>
     <collision>
@@ -226,4 +246,9 @@
           filename="package://wheel_leg3/meshes/link_wheel2.dae" />
       </geometry>
+      <material
+        name="">
+        <color
+          rgba="0.79216 0.81961 0.93333 1" />
+      </material>
     </visual>
     <collision>
@@ -248,5 +273,5 @@
       link="link_wheel2" />
     <axis
-      xyz="0 -1 0" />
+      xyz="0 1 0" />
     <dynamics damping="0.1" friction="0.0"/>
   </joint>

Commit message: 修改base_link转动惯量到计算值

File: wheel-leg_ws/src/wheel_leg3/urdf/wheel_leg3_dae.xacro (robot description, xacro)
@@ -23,18 +23,12 @@
       <mass
         value="3.0" />
-      <!-- <inertia
-        ixx="0.004712"
+      <inertia
+        ixx="0.010361689230147506"
         ixy="-9.6242E-20"
         ixz="2.2781E-20"
-        iyy="0.02081558"
+        iyy="0.0035350575873913923"
         iyz="-2.8504E-20"
-        izz="0.017536" /> -->
-      <inertia
-        ixx="0.02763116"
-        ixy="-9.6242E-20"
-        ixz="2.2781E-20"
-        iyy="0.009424"
-        iyz="-2.8504E-20"
-        izz="0.035072" />
+        izz="0.013152825486630297" />
+      </inertial>
     </inertial>
     <visual>

File: wheel-leg_ws/src/wheel_leg3/urdf/wheel_leg3_stl.xacro (robot description, xacro)
@@ -23,18 +23,11 @@
       <mass
         value="3.0" />
-      <!-- <inertia
-        ixx="0.004712"
+      <inertia
+        ixx="0.010361689230147506"
         ixy="-9.6242E-20"
         ixz="2.2781E-20"
-        iyy="0.02081558"
+        iyy="0.0035350575873913923"
         iyz="-2.8504E-20"
-        izz="0.017536" /> -->
-      <inertia
-        ixx="0.02763116"
-        ixy="-9.6242E-20"
-        ixz="2.2781E-20"
-        iyy="0.009424"
-        iyz="-2.8504E-20"
-        izz="0.035072" />
+        izz="0.013152825486630297" />
     </inertial>
     <visual>
