Commit message: dummy link ->base_footprint，world文件加入到项目文件，rqt_gui视图
机器人位姿真值发布话题/ground_truth/state

File: wheel-leg_ws/src/wheel_leg3/urdf/wheel_leg3_stl.xacro (robot description, xacro)
@@ -7,10 +7,10 @@
   <!-- Import all Gazebo-customization elements, including Gazebo colors -->
   <xacro:include filename="$(find wheel_leg3)/urdf/wheel_leg3.gazebo" />
-  <link name="dummy" />
-  <joint name="joint_dummy_base_link" type="fixed">
+  <link name="base_footprint" />
+  <joint name="joint_base_footprint_base_link" type="fixed">
   <origin
       xyz="0 0 0.253"
       rpy="0 0 0" />
-    <parent link="dummy" />
+    <parent link="base_footprint" />
     <child link="base_link" />
   </joint>

Commit message: 低速下控制ok，速度快后机器人解体

File: wheel-leg_ws/src/wheel_leg3/urdf/wheel_leg3_stl.xacro (robot description, xacro)
@@ -163,4 +163,5 @@
       xyz="0 1 0" />
     <dynamics damping="0.1" friction="0.0"/>
+    <!-- <limit velocity="40.0" effort="10.0" /> -->
   </joint>
   <link
@@ -272,4 +273,5 @@
       xyz="0 1 0" />
     <dynamics damping="0.1" friction="0.0"/>
+    <!-- <limit velocity="40.0" effort="10.0" /> -->
   </joint>
   <link name="imu_link"/>
