Commit message: 解决了腿机构位置控制，但轮腿同时控制会剧烈震荡
猜测轮的驱动力矩使腿部关节抖动，进而导致角速度测量震荡剧烈，控制量也震荡剧烈

File: wheel-leg_ws/src/wheel_leg/urdf/wheel_leg_stl.xacro (robot description, xacro)
@@ -22,5 +22,5 @@
         rpy="0 0 0" />
       <mass
-        value="2" />
+        value="3.0" />
       <inertia
         ixx="0.0104"
@@ -107,10 +107,11 @@
       link="link_right_leg1" />
     <axis
-      xyz="0 0 -1" />
+      xyz="0 0 1" />
     <limit
-      lower="-1.57"
-      upper="1.57"
-      effort="5"
-      velocity="1000" />
+      lower="-1.7"
+      upper="1.7"
+      effort="50"
+      velocity="100" />
+    <dynamics damping="0.1" friction="0.1"/>
   </joint>
   <link
@@ -167,8 +168,9 @@
       xyz="0 0 1" />
     <limit
-      lower="-1.57"
-      upper="1.57"
-      effort="5"
-      velocity="1000" />
+      lower="-1.7"
+      upper="1.7"
+      effort="50"
+      velocity="100" />
+    <dynamics damping="0.1" friction="0.1"/>
   </joint>
   <link
@@ -223,5 +225,5 @@
       link="link_right_wheel" />
     <axis
-      xyz="0 -1 0" />
+      xyz="0 1 0" />
     <dynamics damping="0.1" friction="0.0"/>
   </joint>
@@ -280,8 +282,9 @@
       xyz="0 0 1" />
     <limit
-      lower="-1.57"
-      upper="1.57"
-      effort="5"
-      velocity="1000" />
+      lower="-1.7"
+      upper="1.7"
+      effort="50"
+      velocity="100" />
+    <dynamics damping="0.1" friction="0.1"/>
   </joint>
   <link
@@ -336,10 +339,11 @@
       link="link_left_leg2" />
     <axis
-      xyz="0 0 -1" />
+      xyz="0 0 1" />
     <limit
-      lower="-1.57"
-      upper="1.57"
-      effort="5"
-      velocity="1000" />
+      lower="-1.7"
+      upper="1.7"
+      effort="50"
+      velocity="100" />
+    <dynamics damping="0.1" friction="0.1"/>
   </joint>
   <link
@@ -394,5 +398,5 @@
       link="link_left_wheel" />
     <axis
-      xyz="0 -1 0" />
+      xyz="0 1 0" />
       <dynamics damping="0.1" friction="0.0"/>
   </joint>

Commit message: 通过减小控制参数，改变yaw速度测量解决震荡的问题
初步判断为yaw速度测量震荡导致控制量震荡，导致传感器震荡形成正反馈;根本原因可能是加入活动关节后，某些关节速度测得不准确

File: wheel-leg_ws/src/wheel_leg/urdf/wheel_leg_stl.xacro (robot description, xacro)
@@ -111,7 +111,7 @@
       lower="-1.7"
       upper="1.7"
-      effort="50"
-      velocity="100" />
-    <dynamics damping="0.1" friction="0.1"/>
+      effort="100"
+      velocity="25" />
+    <dynamics damping="0.7" friction="100.0"/>
   </joint>
   <link
@@ -170,7 +170,7 @@
       lower="-1.7"
       upper="1.7"
-      effort="50"
-      velocity="100" />
-    <dynamics damping="0.1" friction="0.1"/>
+      effort="100"
+      velocity="25" />
+    <dynamics damping="0.7" friction="100.0"/>
   </joint>
   <link
@@ -284,7 +284,7 @@
       lower="-1.7"
       upper="1.7"
-      effort="50"
-      velocity="100" />
-    <dynamics damping="0.1" friction="0.1"/>
+      effort="100"
+      velocity="25" />
+    <dynamics damping="0.7" friction="100.0"/>
   </joint>
   <link
@@ -343,7 +343,7 @@
       lower="-1.7"
       upper="1.7"
-      effort="50"
-      velocity="100" />
-    <dynamics damping="0.1" friction="0.1"/>
+      effort="100"
+      velocity="25" />
+    <dynamics damping="0.7" friction="100.0"/>
   </joint>
   <link
@@ -406,5 +406,5 @@
     <parent link="base_link"/>
     <child link="imu_link"/>
-    <origin rpy="0 0 0" xyz="0 0 0.04"/>
+    <origin rpy="0 0 0" xyz="0 0 0"/>
   </joint>
   <transmission name="tran_right_wheel">

Commit message: pid积分抗饱和，机器人碰撞体简化

File: wheel-leg_ws/src/wheel_leg/urdf/wheel_leg_stl.xacro (robot description, xacro)
@@ -50,6 +50,5 @@
         rpy="0 0 0" />
       <geometry>
-        <mesh
-          filename="package://wheel_leg/meshes2/base_link.STL" />
+        <box size="0.12 0.200 0.040"/>
       </geometry>
     </collision>
@@ -88,9 +87,8 @@
     <collision>
       <origin
-        xyz="0 0 0"
-        rpy="0 0 0" />
-      <geometry>
-        <mesh
-          filename="package://wheel_leg/meshes2/link_right_leg1.STL" />
+        xyz="0.065 0.0 0.004"
+        rpy="0 0 0" />
+      <geometry>
+        <box size="0.14 0.015 0.0080"/>
       </geometry>
     </collision>
@@ -147,9 +145,8 @@
     <collision>
       <origin
-        xyz="0 0 0"
-        rpy="0 0 0" />
-      <geometry>
-        <mesh
-          filename="package://wheel_leg/meshes2/link_right_leg2.STL" />
+        xyz="0.065 0.0 -0.004"
+        rpy="0 0 0" />
+      <geometry>
+        <box size="0.14 0.015 0.0080"/>
       </geometry>
     </collision>
@@ -207,8 +204,9 @@
       <origin
         xyz="0 0 0"
-        rpy="0 0 0" />
-      <geometry>
-        <mesh
-          filename="package://wheel_leg/meshes2/link_right_wheel.STL" />
+        rpy="1.57 0 0" />
+      <geometry>
+        <!-- <mesh
+          filename="package://wheel_leg/meshes2/link_right_wheel.STL" /> -->
+        <cylinder length="0.02" radius="0.04"/>
       </geometry>
     </collision>
@@ -261,9 +259,8 @@
     <collision>
       <origin
-        xyz="0 0 0"
-        rpy="0 0 0" />
-      <geometry>
-        <mesh
-          filename="package://wheel_leg/meshes2/link_left_leg1.STL" />
+        xyz="0.065 0.0 -0.004"
+        rpy="0 0 0" />
+      <geometry>
+        <box size="0.14 0.015 0.0080"/>
       </geometry>
     </collision>
@@ -320,9 +317,8 @@
     <collision>
       <origin
-        xyz="0 0 0"
-        rpy="0 0 0" />
-      <geometry>
-        <mesh
-          filename="package://wheel_leg/meshes2/link_left_leg2.STL" />
+        xyz="0.065 0.0 0.004"
+        rpy="0 0 0" />
+      <geometry>
+        <box size="0.14 0.015 0.0080"/>
       </geometry>
     </collision>
@@ -380,8 +376,9 @@
       <origin
         xyz="0 0 0"
-        rpy="0 0 0" />
-      <geometry>
-        <mesh
-          filename="package://wheel_leg/meshes2/link_left_wheel.STL" />
+        rpy="1.57 0 0" />
+      <geometry>
+      <cylinder length="0.02" radius="0.04"/>
+        <!-- <mesh
+          filename="package://wheel_leg/meshes2/link_left_wheel.STL" /> -->
       </geometry>
     </collision>
@@ -408,63 +405,21 @@
     <origin rpy="0 0 0" xyz="0 0 0"/>
   </joint>
-  <transmission name="tran_right_wheel">
-    <type>transmission_interface/SimpleTransmission</type>
-    <joint name="joint_right_leg2_wheel">
-      <hardwareInterface>hardware_interface/EffortJointInterface</hardwareInterface>
-    </joint>
-    <actuator name="motor_right_wheel">
-      <hardwareInterface>hardware_interface/EffortJointInterface</hardwareInterface>
-      <mechanicalReduction>1</mechanicalReduction>
-    </actuator>
-  </transmission>
-  <transmission name="tran_left_wheel">
-    <type>transmission_interface/SimpleTransmission</type>
-    <joint name="joint_left_leg2_wheel">
-      <hardwareInterface>hardware_interface/EffortJointInterface</hardwareInterface>
-    </joint>
-    <actuator name="motor_left_wheel">
-      <hardwareInterface>hardware_interface/EffortJointInterface</hardwareInterface>
-      <mechanicalReduction>1</mechanicalReduction>
-    </actuator>
-  </transmission>
-  <transmission name="tran_base_right_leg1">
-    <type>transmission_interface/SimpleTransmission</type>
-    <joint name="joint_base_right_leg1">
-      <hardwareInterface>hardware_interface/EffortJointInterface</hardwareInterface>
-    </joint>
-    <actuator name="motor_base_right_leg1">
-      <hardwareInterface>hardware_interface/EffortJointInterface</hardwareInterface>
-      <mechanicalReduction>1</mechanicalReduction>
-    </actuator>
-  </transmission>
-  <transmission name="tran_base_left_leg1">
-    <type>transmission_interface/SimpleTransmission</type>
-    <joint name="joint_base_left_leg1">
-      <hardwareInterface>hardware_interface/EffortJointInterface</hardwareInterface>
-    </joint>
-    <actuator name="motor_base_left_leg1">
-      <hardwareInterface>hardware_interface/EffortJointInterface</hardwareInterface>
-      <mechanicalReduction>1</mechanicalReduction>
-    </actuator>
-  </transmission>
-  <transmission name="tran_right_leg1_leg2">
-    <type>transmission_interface/SimpleTransmission</type>
-    <joint name="joint_right_leg1_leg2">
-      <hardwareInterface>hardware_interface/EffortJointInterface</hardwareInterface>
-    </joint>
-    <actuator name="motor_right_leg1_leg2">
-      <hardwareInterface>hardware_interface/EffortJointInterface</hardwareInterface>
-      <mechanicalReduction>1</mechanicalReduction>
-    </actuator>
-  </transmission>
-  <transmission name="tran_left_leg1_leg2">
-    <type>transmission_interface/SimpleTransmission</type>
-    <joint name="joint_left_leg1_leg2">
-      <hardwareInterface>hardware_interface/EffortJointInterface</hardwareInterface>
-    </joint>
-    <actuator name="motor_left_leg1_leg2">
-      <hardwareInterface>hardware_interface/EffortJointInterface</hardwareInterface>
-      <mechanicalReduction>1</mechanicalReduction>
-    </actuator>
-  </transmission>
+  <xacro:macro name="transmission_block" params="joint_name">
+    <transmission name="trans1">
+      <type>transmission_interface/SimpleTransmission</type>
+      <joint name="${joint_name}">
+        <hardwareInterface>hardware_interface/EffortJointInterface</hardwareInterface>
+      </joint>
+      <actuator name="motor1">
+        <hardwareInterface>hardware_interface/EffortJointInterface</hardwareInterface>
+        <mechanicalReduction>1</mechanicalReduction>
+      </actuator>
+    </transmission>
+  </xacro:macro>
+  <xacro:transmission_block joint_name="joint_base_right_leg1"/>
+  <xacro:transmission_block joint_name="joint_base_left_leg1"/>
+  <xacro:transmission_block joint_name="joint_right_leg1_leg2"/>
+  <xacro:transmission_block joint_name="joint_left_leg1_leg2"/>
+  <xacro:transmission_block joint_name="joint_left_leg2_wheel"/>
+  <xacro:transmission_block joint_name="joint_right_leg2_wheel"/>
 </robot>

Commit message: 传感器需要滤波，采用固定关节的情况验证滤波器效果

File: wheel-leg_ws/src/wheel_leg/urdf/wheel_leg_stl.xacro (robot description, xacro)
@@ -96,5 +96,5 @@
   <joint
     name="joint_base_right_leg1"
-    type="revolute">
+    type="fixed">
     <origin
       xyz="0 -0.1 0"
@@ -104,12 +104,4 @@
     <child
       link="link_right_leg1" />
-    <axis
-      xyz="0 0 1" />
-    <limit
-      lower="-1.7"
-      upper="1.7"
-      effort="100"
-      velocity="25" />
-    <dynamics damping="0.7" friction="100.0"/>
   </joint>
   <link
@@ -154,5 +146,5 @@
   <joint
     name="joint_right_leg1_leg2"
-    type="revolute">
+    type="fixed">
     <origin
       xyz="0.13 0 0"
@@ -162,12 +154,4 @@
     <child
       link="link_right_leg2" />
-    <axis
-      xyz="0 0 1" />
-    <limit
-      lower="-1.7"
-      upper="1.7"
-      effort="100"
-      velocity="25" />
-    <dynamics damping="0.7" friction="100.0"/>
   </joint>
   <link
@@ -268,5 +252,5 @@
   <joint
     name="joint_base_left_leg1"
-    type="revolute">
+    type="fixed">
     <origin
       xyz="0 0.1 0"
@@ -276,12 +260,4 @@
     <child
       link="link_left_leg1" />
-    <axis
-      xyz="0 0 1" />
-    <limit
-      lower="-1.7"
-      upper="1.7"
-      effort="100"
-      velocity="25" />
-    <dynamics damping="0.7" friction="100.0"/>
   </joint>
   <link
@@ -326,5 +302,5 @@
   <joint
     name="joint_left_leg1_leg2"
-    type="revolute">
+    type="fixed">
     <origin
       xyz="0.13 0 0"
@@ -334,12 +310,4 @@
     <child
       link="link_left_leg2" />
-    <axis
-      xyz="0 0 1" />
-    <limit
-      lower="-1.7"
-      upper="1.7"
-      effort="100"
-      velocity="25" />
-    <dynamics damping="0.7" friction="100.0"/>
   </joint>
   <link
@@ -417,8 +385,8 @@
     </transmission>
   </xacro:macro>
-  <xacro:transmission_block joint_name="joint_base_right_leg1"/>
+  <!-- <xacro:transmission_block joint_name="joint_base_right_leg1"/>
   <xacro:transmission_block joint_name="joint_base_left_leg1"/>
   <xacro:transmission_block joint_name="joint_right_leg1_leg2"/>
-  <xacro:transmission_block joint_name="joint_left_leg1_leg2"/>
+  <xacro:transmission_block joint_name="joint_left_leg1_leg2"/> -->
   <xacro:transmission_block joint_name="joint_left_leg2_wheel"/>
   <xacro:transmission_block joint_name="joint_right_leg2_wheel"/>

Commit message: 给机器人添加髋关节，但轮子的侧向摩擦力还是会大幅影响腿的形状

File: wheel-leg_ws/src/wheel_leg/urdf/wheel_leg_stl.xacro (robot description, xacro)
@@ -55,4 +55,56 @@
   </link>
   <!-- right -->
+    <link
+    name="link_right_hip">
+    <inertial>
+      <origin
+        xyz="0 0 0"
+        rpy="0 0 0" />
+      <mass
+        value="0.01" />
+      <inertia
+        ixx="1E-5"
+        ixy="0.0"
+        ixz="0.0"
+        iyy="1E-5"
+        iyz="0.0"
+        izz="1E-5" />
+    </inertial>
+    <visual>
+      <origin
+        xyz="0 0 0"
+        rpy="0 0 0" />
+      <geometry>
+        <sphere radius = "0.005"/>
+      </geometry>
+    </visual>
+    <collision>
+      <origin
+        xyz="0 0 0"
+        rpy="0 0 0" />
+      <geometry>
+        <sphere radius = "0.005"/>
+      </geometry>
+    </collision>
+  </link>
+  <joint
+    name="joint_base_right_hip"
+    type="revolute">
+    <origin
+      xyz="0 -0.1 0"
+      rpy="1.5708 1.5708 0" />
+    <parent
+      link="base_link" />
+    <child
+      link="link_right_hip" />
+    <axis
+      xyz="0 -1 0" />
+    <limit
+      lower="-0.524"
+      upper="1.7"
+      effort="100"
+      velocity="25" />
+    <dynamics damping="0.7" friction="100.0"/>
+  </joint>
   <link
     name="link_right_leg1">
@@ -95,11 +147,11 @@
   </link>
   <joint
-    name="joint_base_right_leg1"
+    name="joint_right_hip_right_leg1"
     type="revolute">
     <origin
-      xyz="0 -0.1 0"
-      rpy="1.5708 1.5708 0" />
-    <parent
-      link="base_link" />
+      xyz="0 0 0"
+      rpy="0 0 0" />
+    <parent
+      link="link_right_hip" />
     <child
       link="link_right_leg1" />
@@ -206,6 +258,4 @@
         rpy="1.57 0 0" />
       <geometry>
-        <!-- <mesh
-          filename="package://wheel_leg/meshes2/link_right_wheel.STL" /> -->
         <cylinder length="0.02" radius="0.04"/>
       </geometry>
@@ -227,4 +277,56 @@
   </joint>
   <!-- left -->
+  <link
+    name="link_left_hip">
+    <inertial>
+      <origin
+        xyz="0 0 0"
+        rpy="0 0 0" />
+      <mass
+        value="0.01" />
+      <inertia
+        ixx="1E-5"
+        ixy="0.0"
+        ixz="0.0"
+        iyy="1E-5"
+        iyz="0.0"
+        izz="1E-5" />
+    </inertial>
+    <visual>
+      <origin
+        xyz="0 0 0"
+        rpy="0 0 0" />
+      <geometry>
+        <sphere radius = "0.005"/>
+      </geometry>
+    </visual>
+    <collision>
+      <origin
+        xyz="0 0 0"
+        rpy="0 0 0" />
+      <geometry>
+        <sphere radius = "0.005"/>
+      </geometry>
+    </collision>
+  </link>
+  <joint
+    name="joint_base_left_hip"
+    type="revolute">
+    <origin
+      xyz="0 0.1 0"
+      rpy="1.5708 1.5708 0" />
+    <parent
+      link="base_link" />
+    <child
+      link="link_left_hip" />
+    <axis
+      xyz="0 1 0" />
+    <limit
+      lower="-0.524"
+      upper="1.7"
+      effort="100"
+      velocity="25" />
+    <dynamics damping="0.7" friction="100.0"/>
+  </joint>
   <link
     name="link_left_leg1">
@@ -267,11 +369,11 @@
   </link>
   <joint
-    name="joint_base_left_leg1"
+    name="joint_left_hip_left_leg1"
     type="revolute">
     <origin
-      xyz="0 0.1 0"
-      rpy="1.5708 1.5708 0" />
-    <parent
-      link="base_link" />
+      xyz="0 0 0"
+      rpy="0 0 0" />
+    <parent
+      link="link_left_hip" />
     <child
       link="link_left_leg1" />
@@ -417,6 +519,8 @@
     </transmission>
   </xacro:macro>
-  <xacro:transmission_block joint_name="joint_base_right_leg1"/>
-  <xacro:transmission_block joint_name="joint_base_left_leg1"/>
+  <xacro:transmission_block joint_name="joint_base_right_hip"/>
+  <xacro:transmission_block joint_name="joint_right_hip_right_leg1"/>
+  <xacro:transmission_block joint_name="joint_base_left_hip"/>
+  <xacro:transmission_block joint_name="joint_left_hip_left_leg1"/>
   <xacro:transmission_block joint_name="joint_right_leg1_leg2"/>
   <xacro:transmission_block joint_name="joint_left_leg1_leg2"/>

Commit message: 为机器人加入膝关节

File: wheel-leg_ws/src/wheel_leg/urdf/wheel_leg_stl.xacro (robot description, xacro)
@@ -105,5 +105,5 @@
       effort="100"
       velocity="25" />
-    <dynamics damping="0.7" friction="100.0"/>
+    <dynamics damping="0.7" friction="1.0"/>
   </joint>
   <link
@@ -163,5 +163,57 @@
       effort="100"
       velocity="25" />
-    <dynamics damping="0.7" friction="100.0"/>
+    <dynamics damping="0.7" friction="1.0"/>
+  </joint>
+  <link
+    name="link_right_knee">
+    <inertial>
+      <origin
+        xyz="0 0 0"
+        rpy="0 0 0" />
+      <mass
+        value="0.01" />
+      <inertia
+        ixx="1E-5"
+        ixy="0.0"
+        ixz="0.0"
+        iyy="1E-5"
+        iyz="0.0"
+        izz="1E-5" />
+    </inertial>
+    <visual>
+      <origin
+        xyz="0 0 0"
+        rpy="0 0 0" />
+      <geometry>
+        <sphere radius = "0.005"/>
+      </geometry>
+    </visual>
+    <collision>
+      <origin
+        xyz="0 0 0"
+        rpy="0 0 0" />
+      <geometry>
+        <sphere radius = "0.005"/>
+      </geometry>
+    </collision>
+  </link>
+  <joint
+    name="joint_right_leg1_knee"
+    type="revolute">
+    <origin
+      xyz="0.13 0 0"
+      rpy="0 0 0" />
+    <parent
+      link="link_right_leg1" />
+    <child
+      link="link_right_knee" />
+    <axis
+      xyz="0 -1 0" />
+    <limit
+      lower="-1.7"
+      upper="1.7"
+      effort="100"
+      velocity="25" />
+    <dynamics damping="0.7" friction="1.0"/>
   </joint>
   <link
@@ -205,11 +257,11 @@
   </link>
   <joint
-    name="joint_right_leg1_leg2"
-    type="revolute">
-    <origin
-      xyz="0.13 0 0"
+    name="joint_right_knee_leg2"
+    type="revolute">
+    <origin
+      xyz="0.0 0 0"
       rpy="0 0 0" />
     <parent
-      link="link_right_leg1" />
+      link="link_right_knee" />
     <child
       link="link_right_leg2" />
@@ -221,5 +273,5 @@
       effort="100"
       velocity="25" />
-    <dynamics damping="0.7" friction="100.0"/>
+    <dynamics damping="0.7" friction="1.0"/>
   </joint>
   <link
@@ -327,5 +379,5 @@
       effort="100"
       velocity="25" />
-    <dynamics damping="0.7" friction="100.0"/>
+    <dynamics damping="0.7" friction="1.0"/>
   </joint>
   <link
@@ -385,5 +437,57 @@
       effort="100"
       velocity="25" />
-    <dynamics damping="0.7" friction="100.0"/>
+    <dynamics damping="0.7" friction="1.0"/>
+  </joint>
+  <link
+    name="link_left_knee">
+    <inertial>
+      <origin
+        xyz="0 0 0"
+        rpy="0 0 0" />
+      <mass
+        value="0.01" />
+      <inertia
+        ixx="1E-5"
+        ixy="0.0"
+        ixz="0.0"
+        iyy="1E-5"
+        iyz="0.0"
+        izz="1E-5" />
+    </inertial>
+    <visual>
+      <origin
+        xyz="0 0 0"
+        rpy="0 0 0" />
+      <geometry>
+        <sphere radius = "0.005"/>
+      </geometry>
+    </visual>
+    <collision>
+      <origin
+        xyz="0 0 0"
+        rpy="0 0 0" />
+      <geometry>
+        <sphere radius = "0.005"/>
+      </geometry>
+    </collision>
+  </link>
+  <joint
+    name="joint_left_leg1_knee"
+    type="revolute">
+    <origin
+      xyz="0.13 0 0"
+      rpy="0 0 0" />
+    <parent
+      link="link_left_leg1" />
+    <child
+      link="link_left_knee" />
+    <axis
+      xyz="0 1 0" />
+    <limit
+      lower="-1.7"
+      upper="1.7"
+      effort="100"
+      velocity="25" />
+    <dynamics damping="0.7" friction="1.0"/>
   </joint>
   <link
@@ -427,11 +531,11 @@
   </link>
   <joint
-    name="joint_left_leg1_leg2"
-    type="revolute">
-    <origin
-      xyz="0.13 0 0"
+    name="joint_left_knee_leg2"
+    type="revolute">
+    <origin
+      xyz="0.0 0 0"
       rpy="0 0 0" />
     <parent
-      link="link_left_leg1" />
+      link="link_left_knee" />
     <child
       link="link_left_leg2" />
@@ -443,5 +547,5 @@
       effort="100"
       velocity="25" />
-    <dynamics damping="0.7" friction="100.0"/>
+    <dynamics damping="0.7" friction="1.0"/>
   </joint>
   <link
@@ -480,7 +584,5 @@
         rpy="1.57 0 0" />
       <geometry>
-      <cylinder length="0.02" radius="0.04"/>
-        <!-- <mesh
-          filename="package://wheel_leg/meshes2/link_left_wheel.STL" /> -->
+        <cylinder length="0.02" radius="0.04"/>
       </geometry>
     </collision>
@@ -523,6 +625,8 @@
   <xacro:transmission_block joint_name="joint_base_left_hip"/>
   <xacro:transmission_block joint_name="joint_left_hip_left_leg1"/>
-  <xacro:transmission_block joint_name="joint_right_leg1_leg2"/>
-  <xacro:transmission_block joint_name="joint_left_leg1_leg2"/>
+  <xacro:transmission_block joint_name="joint_right_leg1_knee"/>
+  <xacro:transmission_block joint_name="joint_right_knee_leg2"/>
+  <xacro:transmission_block joint_name="joint_left_leg1_knee"/>
+  <xacro:transmission_block joint_name="joint_left_knee_leg2"/>
   <xacro:transmission_block joint_name="joint_left_leg2_wheel"/>
   <xacro:transmission_block joint_name="joint_right_leg2_wheel"/>

Commit message: 添加激光雷达

File: wheel-leg_ws/src/wheel_leg/urdf/wheel_leg_stl.xacro (robot description, xacro)
@@ -5,4 +5,6 @@
 <robot
   name="wheel_leg" xmlns:xacro="http://www.ros.org/wiki/xacro">
+  <xacro:include filename="$(find wheel_leg)/urdf/sick_tim.urdf.xacro" />
+  <xacro:rplidarA2 name="laser" ros_topic="scan"   />
   <!-- Import all Gazebo-customization elements, including Gazebo colors -->
   <xacro:include filename="$(find wheel_leg)/urdf/wheel_leg.gazebo" />
@@ -608,4 +610,11 @@
     <child link="imu_link"/>
     <origin rpy="0 0 0" xyz="0 0 0"/>
+  </joint>
+  <link name="laser_mount_link"/>
+  <joint name="base_to_laser" type="fixed">
+    <axis rpy="0 0 0" xyz="0 0 0"/>
+    <parent link="base_link"/>
+    <child link="laser_mount_link"/>
+    <origin rpy="0 0 0" xyz="0 0 0.04"/>
   </joint>
   <xacro:macro name="transmission_block" params="joint_name">
